File: PCB/watch.brd (EAGLE design)
At the start: 81.1 x 53.1 mm, 58 parts, among them IC1 ISL1209, J2 USB-MICROB, Q1 32.768 KHz, T1 BC850, U2 MKL27Z256VLH4

Commit message: fixed some fuck ups
Routing:
- net PTD1: track 73.4 -> 49.8 mm, vias 0 -> 1
- net GND: track 53.2 -> 73.9 mm, vias 4 -> 7
Changed lines of the file:
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@@
 <wire x1="70.231" y1="43.434" x2="70.231" y2="43.395" width="0.254" layer="1"/>
 <wire x1="70.231" y1="43.395" x2="68.834" y2="41.998" width="0.254" layer="1"/>
-<wire x1="72.51" y1="34.35" x2="66.868" y2="32.579" width="0" layer="19" extent="1-16"/>
+<wire x1="66.868" y1="32.579" x2="66.675" y2="32.386" width="0.254" layer="16"/>
+<wire x1="66.675" y1="32.386" x2="66.675" y2="31.496" width="0.254" layer="16"/>
+<via x="66.675" y="31.496" extent="1-16" drill="0.6"/>
+<wire x1="66.675" y1="31.496" x2="67.056" y2="31.115" width="0.254" layer="1"/>
+<wire x1="67.056" y1="31.115" x2="67.056" y2="25.908" width="0.254" layer="1"/>
+<wire x1="67.056" y1="25.908" x2="65.913" y2="24.765" width="0.254" layer="1"/>
+<wire x1="65.913" y1="24.765" x2="65.786" y2="24.765" width="0.254" layer="1"/>
+<via x="65.786" y="24.765" extent="1-16" drill="0.6"/>
+<wire x1="65.786" y1="24.765" x2="64.643" y2="23.622" width="0.254" layer="16"/>
+<wire x1="64.643" y1="23.622" x2="64.643" y2="19.939" width="0.254" layer="16"/>
+<wire x1="64.643" y1="19.939" x2="69.215" y2="19.939" width="0.254" layer="16"/>
+<wire x1="69.215" y1="19.939" x2="69.215" y2="21.971" width="0.254" layer="16"/>
+<via x="69.215" y="21.971" extent="1-16" drill="0.6"/>
+<wire x1="69.215" y1="21.971" x2="69.342" y2="22.098" width="0.254" layer="1"/>
+<wire x1="60.325" y1="44.069" x2="56.94858125" y2="40.23061875" width="0" layer="19" extent="1-16"/>
 <wire x1="76.611" y1="52.578" x2="79.121" y2="51.601" width="0" layer="19" extent="1-1"/>
-<wire x1="86.741" y1="47.435" x2="87.51" y2="43.35" width="0" layer="19" extent="1-1"/>
-<wire x1="56.94858125" y1="40.23061875" x2="60.325" y2="44.069" width="0" layer="19" extent="1-16"/>
 <wire x1="48.99361875" y1="35.634415625" x2="56.94858125" y2="40.23061875" width="0" layer="19" extent="1-1"/>
 <wire x1="48.286515625" y1="47.478475" x2="58.674" y2="45.72" width="0" layer="19" extent="1-16"/>
@@
 <contactref element="U2" pad="58"/>
 <contactref element="LED-W" pad="A"/>
-<wire x1="75.565" y1="18.669" x2="82.423" y2="25.527" width="0.254" layer="1"/>
-<wire x1="82.423" y1="25.527" x2="82.423" y2="28.829" width="0.254" layer="1"/>
-<wire x1="82.423" y1="28.829" x2="83.058" y2="29.464" width="0.254" layer="1"/>
-<wire x1="83.058" y1="29.464" x2="88.519" y2="29.464" width="0.254" layer="1"/>
-<wire x1="88.519" y1="29.464" x2="89.408" y2="30.353" width="0.254" layer="1"/>
-<wire x1="89.408" y1="30.353" x2="89.408" y2="45.974" width="0.254" layer="1"/>
-<wire x1="89.408" y1="45.974" x2="89.281" y2="46.101" width="0.254" layer="1"/>
-<wire x1="89.281" y1="46.101" x2="70.358" y2="46.101" width="0.254" layer="1"/>
-<wire x1="70.358" y1="46.101" x2="68.072" y2="48.387" width="0.254" layer="1"/>
+<wire x1="70.739" y1="45.72" x2="68.072" y2="48.387" width="0.254" layer="1"/>
 <wire x1="68.072" y1="48.387" x2="56.007" y2="48.387" width="0.254" layer="1"/>
 <wire x1="56.007" y1="48.387" x2="54.120140625" y2="46.500140625" width="0.254" layer="1"/>
 <wire x1="54.120140625" y1="46.500140625" x2="54.120140625" y2="46.41781875" width="0.254" layer="1"/>
+<wire x1="70.739" y1="45.72" x2="73.787" y2="45.72" width="0.254" layer="1"/>
+<wire x1="75.565" y1="18.669" x2="75.819" y2="18.669" width="0.254" layer="16"/>
+<wire x1="75.819" y1="18.669" x2="75.819" y2="43.688" width="0.254" layer="16"/>
+<via x="75.819" y="43.688" extent="1-16" drill="0.6"/>
+<wire x1="75.819" y1="43.688" x2="73.787" y2="45.72" width="0.254" layer="1"/>
 </signal>
 <signal name="N$39">

Commit message: moar refactoring
Routing:
- net GND: track 73.9 -> 80.2 mm, vias 7 -> 9
- net PTA3: track 39.8 -> 33.6 mm
Changed lines of the file:
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@@
 <via x="69.215" y="21.971" extent="1-16" drill="0.6"/>
 <wire x1="69.215" y1="21.971" x2="69.342" y2="22.098" width="0.254" layer="1"/>
+<wire x1="79.121" y1="51.601" x2="79.121" y2="49.53" width="0.254" layer="1"/>
+<via x="79.121" y="49.53" extent="1-16" drill="0.6"/>
+<wire x1="79.121" y1="49.53" x2="77.851" y2="50.8" width="0.254" layer="16"/>
+<wire x1="77.851" y1="50.8" x2="77.597" y2="50.8" width="0.254" layer="16"/>
+<via x="77.597" y="50.8" extent="1-16" drill="0.6"/>
+<wire x1="77.597" y1="50.8" x2="76.415" y2="50.8" width="0.254" layer="1"/>
+<wire x1="76.415" y1="50.8" x2="76.415" y2="49.784" width="0.254" layer="1"/>
 <wire x1="60.325" y1="44.069" x2="56.94858125" y2="40.23061875" width="0" layer="19" extent="1-16"/>
-<wire x1="76.611" y1="52.578" x2="79.121" y2="51.601" width="0" layer="19" extent="1-1"/>
 <wire x1="48.99361875" y1="35.634415625" x2="56.94858125" y2="40.23061875" width="0" layer="19" extent="1-1"/>
 <wire x1="48.286515625" y1="47.478475" x2="58.674" y2="45.72" width="0" layer="19" extent="1-16"/>
@@
 <contactref element="SWD_BREAKOUT" pad="SWD_CLK"/>
 <contactref element="U2" pad="22"/>
-<wire x1="26.035" y1="54.483" x2="33.655" y2="46.863" width="0.254" layer="16"/>
-<wire x1="33.655" y1="46.863" x2="51.308" y2="46.863" width="0.254" layer="16"/>
-<via x="51.308" y="46.863" extent="1-16" drill="0.6"/>
-<wire x1="51.308" y1="46.863" x2="51.308" y2="44.31278125" width="0.254" layer="1"/>
-<wire x1="51.308" y1="44.31278125" x2="45.811628125" y2="38.816409375" width="0.254" layer="1"/>
+<wire x1="26.035" y1="54.483" x2="29.464" y2="54.483" width="0.254" layer="16"/>
+<wire x1="29.464" y1="54.483" x2="37.338" y2="46.609" width="0.254" layer="16"/>
+<wire x1="37.338" y1="46.609" x2="51.054" y2="46.609" width="0.254" layer="16"/>
+<wire x1="51.054" y1="46.609" x2="51.181" y2="46.482" width="0.254" layer="16"/>
+<via x="51.181" y="46.482" extent="1-16" drill="0.6"/>
+<wire x1="51.181" y1="46.482" x2="51.181" y2="44.18578125" width="0.254" layer="1"/>
+<wire x1="51.181" y1="44.18578125" x2="45.811628125" y2="38.816409375" width="0.254" layer="1"/>
 </signal>
 <signal name="PTA3">
 <contactref element="U2" pad="25"/>
 <contactref element="SWD_BREAKOUT" pad="SWD_DIO"/>
-<wire x1="26.035" y1="51.943" x2="26.924" y2="51.943" width="0.254" layer="16"/>
-<wire x1="26.924" y1="51.943" x2="35.306" y2="43.561" width="0.254" layer="16"/>
-<wire x1="35.306" y1="43.561" x2="51.435" y2="43.561" width="0.254" layer="16"/>
-<wire x1="51.435" y1="43.561" x2="52.578" y2="44.704" width="0.254" layer="16"/>
-<via x="52.578" y="44.704" extent="1-16" drill="0.6"/>
-<wire x1="46.8722875" y1="37.75575" x2="50.673" y2="41.5564625" width="0.254" layer="1"/>
-<wire x1="50.673" y1="41.5564625" x2="50.673" y2="42.545" width="0.254" layer="1"/>
-<wire x1="50.673" y1="42.545" x2="52.578" y2="44.45" width="0.254" layer="1"/>
-<wire x1="52.578" y1="44.45" x2="52.578" y2="44.704" width="0.254" layer="1"/>
+<wire x1="26.035" y1="51.943" x2="30.734" y2="47.244" width="0.254" layer="16"/>
+<wire x1="30.734" y1="47.244" x2="31.623" y2="47.244" width="0.254" layer="16"/>
+<wire x1="31.623" y1="47.244" x2="36.957" y2="41.91" width="0.254" layer="16"/>
+<wire x1="36.957" y1="41.91" x2="50.038" y2="41.91" width="0.254" layer="16"/>
+<via x="50.038" y="41.91" extent="1-16" drill="0.6"/>
+<wire x1="50.038" y1="41.91" x2="49.911" y2="40.7944625" width="0.254" layer="1"/>
+<wire x1="49.911" y1="40.7944625" x2="46.8722875" y2="37.75575" width="0.254" layer="1"/>
 </signal>
 <signal name="N$3">

Commit message: fixed more wiring issues. started i2c
Routing:
- net PTC8: track 6.56 -> 44.0 mm, vias 0 -> 2
- net GND: track 80.2 -> 97.2 mm, vias 9 -> 11
- net V+: track 49.4 -> 60.1 mm, vias 6 -> 7
- net N$1: track 0.00 -> 10.6 mm
- net PTC0: track 57.5 -> 60.0 mm
Changed lines of the file:
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@@
 <contactref element="U$1" pad="22"/>
 <contactref element="U$1" pad="35"/>
-<wire x1="25.334525" y1="33.104853125" x2="24.366259375" y2="41.610290625" width="0" layer="19" extent="1-1"/>
+<wire x1="24.366259375" y1="41.610290625" x2="22.352" y2="39.59603125" width="0.254" layer="1"/>
+<wire x1="22.352" y1="39.59603125" x2="22.352" y2="36.087378125" width="0.254" layer="1"/>
+<wire x1="22.352" y1="36.087378125" x2="25.334525" y2="33.104853125" width="0.254" layer="1"/>
 </signal>
 <signal name="GND">
@@
 <wire x1="77.597" y1="50.8" x2="76.415" y2="50.8" width="0.254" layer="1"/>
 <wire x1="76.415" y1="50.8" x2="76.415" y2="49.784" width="0.254" layer="1"/>
+<wire x1="27.6945875" y1="38.15164375" x2="26.416" y2="36.87305625" width="0.254" layer="1"/>
+<wire x1="26.416" y1="36.87305625" x2="26.416" y2="35.56" width="0.254" layer="1"/>
+<wire x1="26.416" y1="35.56" x2="27.063846875" y2="34.912153125" width="0.254" layer="1"/>
+<wire x1="27.063846875" y1="34.912153125" x2="27.063846875" y2="34.769015625" width="0.254" layer="1"/>
+<wire x1="18.19495625" y1="40.80095625" x2="17.145" y2="39.751" width="0.254" layer="1"/>
+<wire x1="17.145" y1="39.751" x2="17.145" y2="39.497" width="0.254" layer="1"/>
+<via x="17.145" y="39.497" extent="1-16" drill="0.6"/>
+<wire x1="17.145" y1="39.497" x2="21.209" y2="35.433" width="0.254" layer="16"/>
+<wire x1="21.209" y1="35.433" x2="24.257" y2="35.433" width="0.254" layer="16"/>
+<via x="24.257" y="35.433" extent="1-16" drill="0.6"/>
+<wire x1="24.257" y1="35.433" x2="26.289" y2="35.433" width="0.254" layer="1"/>
+<wire x1="26.289" y1="35.433" x2="26.416" y2="35.56" width="0.254" layer="1" curve="90"/>
 <wire x1="60.325" y1="44.069" x2="56.94858125" y2="40.23061875" width="0" layer="19" extent="1-16"/>
 <wire x1="48.99361875" y1="35.634415625" x2="56.94858125" y2="40.23061875" width="0" layer="19" extent="1-1"/>
@@
 <wire x1="20.9619125" y1="41.109865625" x2="21.59" y2="40.481778125" width="0.3048" layer="1"/>
 <wire x1="21.59" y1="40.481778125" x2="21.59" y2="39.07294375" width="0.3048" layer="1"/>
-<wire x1="21.59" y1="39.07294375" x2="20.087528125" y2="37.570471875" width="0.3048" layer="1"/>
-<wire x1="20.087528125" y1="37.570471875" x2="18.025409375" y2="35.508353125" width="0.3048" layer="1"/>
-<wire x1="24.758084375" y1="32.55013125" x2="24.758084375" y2="32.899915625" width="0.3048" layer="1"/>
-<wire x1="24.758084375" y1="32.899915625" x2="20.087528125" y2="37.570471875" width="0.3048" layer="1"/>
+<wire x1="21.59" y1="39.07294375" x2="19.960528125" y2="37.443471875" width="0.3048" layer="1"/>
+<wire x1="19.960528125" y1="37.443471875" x2="18.025409375" y2="35.508353125" width="0.3048" layer="1"/>
 <wire x1="64.94" y1="42.86" x2="65.382" y2="42.799" width="0.254" layer="1"/>
 <wire x1="61.8949" y1="44.974" x2="62.611" y2="44.2579" width="0.254" layer="1"/>
@@
 <wire x1="63.373" y1="42.926" x2="64.874" y2="42.926" width="0.254" layer="1"/>
 <wire x1="64.874" y1="42.926" x2="64.94" y2="42.86" width="0.254" layer="1"/>
+<wire x1="26.162" y1="43.776" x2="27.774" y2="43.776" width="0.254" layer="1"/>
+<wire x1="27.774" y1="43.776" x2="27.94" y2="43.942" width="0.254" layer="1"/>
+<via x="27.94" y="43.942" extent="1-16" drill="0.6"/>
+<wire x1="27.94" y1="43.942" x2="28.702" y2="44.704" width="0.254" layer="16"/>
+<wire x1="24.758084375" y1="32.55013125" x2="19.960528125" y2="37.3476875" width="0.254" layer="1"/>
+<wire x1="19.960528125" y1="37.3476875" x2="19.960528125" y2="37.443471875" width="0.254" layer="1"/>
+<wire x1="24.758084375" y1="32.55013125" x2="25.304215625" y2="32.004" width="0.254" layer="1"/>
+<wire x1="25.304215625" y1="32.004" x2="28.067" y2="32.004" width="0.254" layer="1"/>
+<wire x1="28.067" y1="32.004" x2="30.353" y2="34.29" width="0.254" layer="1"/>
+<wire x1="30.353" y1="34.29" x2="30.353" y2="35.433" width="0.254" layer="1"/>
 <wire x1="45.104521875" y1="44.29648125" x2="48.640065625" y2="47.832028125" width="0" layer="19" extent="1-1"/>
 <wire x1="48.640065625" y1="35.98796875" x2="45.104521875" y2="44.29648125" width="0" layer="19" extent="1-1"/>
@@
 <wire x1="60.706" y1="44.958" x2="57.302134375" y2="40.584171875" width="0" layer="19" extent="1-16"/>
 <wire x1="17.78" y1="45.3" x2="19.939" y2="42.545" width="0" layer="19" extent="1-1"/>
-<wire x1="20.32" y1="48.26" x2="17.78" y2="45.3" width="0" layer="19" extent="1-1"/>
-<wire x1="29.718" y1="35.052" x2="24.758084375" y2="32.899915625" width="0" layer="19" extent="1-1"/>
-<wire x1="26.162" y1="43.776" x2="21.59" y2="40.481778125" width="0" layer="19" extent="1-1"/>
 <wire x1="41.822" y1="16.002" x2="48.640065625" y2="35.98796875" width="0" layer="19" extent="1-1"/>
 <wire x1="43.649" y1="13.335" x2="41.822" y2="16.002" width="0" layer="19" extent="1-1"/>
@@
 <wire x1="-63.92" y1="73.66" x2="-60.11" y2="73.66" width="0" layer="19" extent="1-1"/>
 <wire x1="-67.73" y1="73.66" x2="-63.92" y2="73.66" width="0" layer="19" extent="1-1"/>
+<wire x1="20.32" y1="48.26" x2="17.78" y2="45.3" width="0" layer="19" extent="1-1"/>
 </signal>
 <signal name="PTA19">
@@
 <wire x1="61.8949" y1="45.974" x2="57.2118875" y2="45.974" width="0.254" layer="1"/>
 <wire x1="57.2118875" y1="45.974" x2="55.887921875" y2="44.650034375" width="0.254" layer="1"/>
-<wire x1="26.162" y1="42.076" x2="55.887921875" y2="44.650034375" width="0" layer="19" extent="1-1"/>
-<wire x1="26.030421875" y1="39.880965625" x2="26.162" y2="42.076" width="0" layer="19" extent="1-1"/>
+<wire x1="26.162" y1="42.076" x2="26.162" y2="41.275" width="0.254" layer="1"/>
+<wire x1="26.162" y1="41.275" x2="26.797" y2="40.64" width="0.254" layer="1"/>
+<wire x1="26.797" y1="40.64" x2="26.78945625" y2="40.64" width="0.254" layer="1"/>
+<wire x1="26.78945625" y1="40.64" x2="26.030421875" y2="39.880965625" width="0.254" layer="1"/>
+<wire x1="26.797" y1="40.64" x2="30.988" y2="40.64" width="0.254" layer="1"/>
+<wire x1="30.988" y1="40.64" x2="33.02" y2="38.608" width="0.254" layer="1"/>
+<wire x1="33.02" y1="38.608" x2="38.481" y2="38.608" width="0.254" layer="1"/>
+<via x="38.481" y="38.608" extent="1-16" drill="0.6"/>
+<wire x1="38.481" y1="38.608" x2="51.181" y2="38.608" width="0.254" layer="16"/>
+<wire x1="51.181" y1="38.608" x2="51.435" y2="38.354" width="0.254" layer="16"/>
+<wire x1="51.435" y1="38.354" x2="52.451" y2="38.354" width="0.254" layer="16"/>
+<wire x1="52.451" y1="38.354" x2="53.975" y2="39.878" width="0.254" layer="16"/>
+<wire x1="53.975" y1="39.878" x2="53.975" y2="43.307" width="0.254" layer="16"/>
+<via x="53.975" y="43.307" extent="1-16" drill="0.6"/>
+<wire x1="53.975" y1="43.307" x2="54.5448875" y2="43.307" width="0.254" layer="1"/>
+<wire x1="54.5448875" y1="43.307" x2="55.887921875" y2="44.650034375" width="0.254" layer="1"/>
 </signal>
 <signal name="PTC9">
@@
 <wire x1="61.8949" y1="46.474" x2="57.00478125" y2="46.474" width="0.254" layer="1"/>
 <wire x1="57.00478125" y1="46.474" x2="55.53436875" y2="45.0035875" width="0.254" layer="1"/>
+<wire x1="17.78" y1="43.6" x2="23.8115375" y2="42.18673125" width="0" layer="19" extent="1-1"/>
 <wire x1="23.8115375" y1="42.18673125" x2="55.53436875" y2="45.0035875" width="0" layer="19" extent="1-1"/>
-<wire x1="17.78" y1="43.6" x2="23.8115375" y2="42.18673125" width="0" layer="19" extent="1-1"/>
 </signal>
 <signal name="PTE20">
@@
 <wire x1="27.178" y1="32.609" x2="27.178" y2="41.021" width="0.3048" layer="16"/>
 <wire x1="27.178" y1="41.021" x2="51.562" y2="41.021" width="0.3048" layer="16"/>
-<wire x1="51.562" y1="41.021" x2="51.562" y2="43.053" width="0.3048" layer="16"/>
-<wire x1="51.562" y1="43.053" x2="54.737" y2="43.053" width="0.3048" layer="16"/>
-<wire x1="54.737" y1="43.053" x2="54.737" y2="41.021" width="0.3048" layer="16"/>
+<wire x1="51.562" y1="41.021" x2="51.562" y2="44.323" width="0.3048" layer="16"/>
+<wire x1="51.562" y1="44.323" x2="54.737" y2="44.323" width="0.3048" layer="16"/>
+<wire x1="54.737" y1="44.323" x2="54.737" y2="41.021" width="0.3048" layer="16"/>
 <via x="54.737" y="41.021" extent="1-16" drill="0.6"/>
 <wire x1="54.737" y1="41.021" x2="54.737" y2="39.613778125" width="0.3048" layer="1"/>
